Commit message: Add visualization option for non-simplified paths and observation points

File: models/warehouse_no_ground/model.urdf (robot description, URDF)
Before this commit: robot warehouse, 1 links, 0 joints
Links:
- link base: geometry collision mesh filename=../models/warehouse_no_ground/model.dae scale=1.00000 1.00000 1.00000; visual mesh filename=../models/warehouse_no_ground/model.dae scale=1.00000 1.00000 1.00000
