Commit message: Update camera state sampler to work with all environments

File: models/car/car.urdf (robot description, URDF)
Before this commit: robot car, 2 links, 1 joints
Joints:
- joint base_to_camera: axis (none) -> 0 0 1; type fixed -> continuous

File: models/create_description/urdf/create_2.urdf (robot description, URDF)
Before this commit: robot create_2, 12 links, 11 joints
Joints:
- joint camera_joint: axis 1 0 0 -> 0 0 1; type fixed -> continuous
- joint left_wheel_joint: type continuous -> fixed
- joint right_wheel_joint: type continuous -> fixed
