Commit message: Add sampling of good camera positions

File: examples/combined.urdf (robot description, URDF)
Before this commit: robot create_2, 22 links, 21 joints
Joints:
- joint left_wheel_joint: type continuous -> fixed
- joint panda_joint3: type revolute -> fixed
- joint panda_joint4: type revolute -> fixed
- joint panda_joint5: type revolute -> fixed
- joint panda_joint7: type revolute -> fixed
- joint right_wheel_joint: type continuous -> fixed

Commit message: Add camera state sampler

File: examples/combined.urdf (robot description, URDF)
Before this commit: robot create_2, 22 links, 21 joints
Joints:
- joint panda_joint3: type fixed -> revolute
- joint panda_joint4: type fixed -> revolute
- joint panda_joint5: type fixed -> revolute
- joint panda_joint7: type fixed -> revolute

Commit message: Fix self-collision of mobile_arm

File: examples/combined.urdf (robot description, URDF)
Before this commit: robot create_2, 22 links, 21 joints
Joints:
- joint joint_dummy1: origin xyz=0.00000 0.00000 0.00000 rpy=0.00000 0.00000 0.00000 -> xyz=0.00000 0.00000 0.5 rpy=0.00000 0.00000 0.00000

File: models/car/car.urdf (robot description, URDF)
Before this commit: robot car, 2 links, 1 joints
Links:
- link base: geometry collision box size=0.5 0.3 0.1; visual box size=0.5 0.3 0.1
