Commit message: Add simple search and rescue environment

File: models/office_simple/office.urdf (robot description, URDF)
Before this commit: robot office, 1 links, 0 joints
Links:
- link base: geometry collision mesh filename=package://office_simple/office.obj scale=0.4 0.4 0.4; visual mesh filename=package://office_simple/office.obj scale=0.4 0.4 0.4

File: models/warehouse_no_ground/warehouse_observation_point.urdf (robot description, URDF)
Before this commit: robot warehouse, 1 links, 0 joints
Links:
- link base: geometry collision mesh filename=../models/warehouse_no_ground/warehouse_observation_point.o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 scale=1.00000 1.00000 1.00000; visual mesh filename=../models/warehouse_no_ground/warehouse_observation_point.o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 scale=1.00000 1.00000 1.00000
