Commit message: Add door environment

File: models/floor_plan/floor_plan.urdf (robot description, URDF)
Before this commit: robot house, 1 links, 0 joints
Links:
- link base: geometry collision mesh filename=package://floor_plan/floor_plan.obj scale=0.4 0.4 0.4; visual mesh filename=package://floor_plan/floor_plan.obj scale=0.4 0.4 0.4

File: models/house/door.urdf (robot description, URDF)
Before this commit: robot house, 1 links, 0 joints
Links:
- link base: geometry collision mesh filename=package://floor_plan/door.obj scale=0.4 0.4 0.4; visual mesh filename=package://floor_plan/door.obj scale=0.4 0.4 0.4

Commit message: Add extended door demo

File: models/floor_plan/floor_plan.urdf (robot description, URDF)
Before this commit: robot floor_plan, 1 links, 0 joints
Links:
- link base: geometry collision mesh filename=package://floor_plan/floor_plan_extended.obj scale=0.4 0.4 0.4; visual mesh filename=package://floor_plan/floor_plan_extended.obj scale=0.4 0.4 0.4
